Commit message: 动态清除过期障碍物点云

File: tcpa_sim_env/urdf/robot.xacro (robot description, xacro)
@@ -100,4 +100,31 @@
     <origin xyz="0.0 0.0 ${base_height / 2.0 + imu_size / 2.0}" rpy="0 0 0"/>
   </joint>
+  <link name="nav_scan_frame">
+    <visual>
+      <origin xyz="0 0 0" rpy="0 0 0"/>
+      <geometry>
+        <cylinder radius="0.04" length="0.04"/>
+      </geometry>
+      <material name="nav_scan_green">
+        <color rgba="0.10 0.75 0.20 1.0"/>
+      </material>
+    </visual>
+    <collision>
+      <origin xyz="0 0 0" rpy="0 0 0"/>
+      <geometry>
+        <cylinder radius="0.04" length="0.04"/>
+      </geometry>
+    </collision>
+    <inertial>
+      <origin xyz="0 0 0" rpy="0 0 0"/>
+      <mass value="0.05"/>
+      <inertia ixx="5e-5" ixy="0.0" ixz="0.0" iyy="5e-5" iyz="0.0" izz="5e-5"/>
+    </inertial>
+  </link>
+  <joint name="nav_scan_joint" type="fixed">
+    <parent link="base_link"/>
+    <child link="nav_scan_frame"/>
+    <origin xyz="0.0 0.0 ${base_height / 2.0 + 0.03}" rpy="0 0 0"/>
+  </joint>
   <gazebo reference="base_link">
     <material>Gazebo/Gray</material>
@@ -144,4 +171,39 @@
     </xacro:mid360>
   </xacro:if>
+  <gazebo reference="nav_scan_frame">
+    <sensor name="nav_scan_sensor" type="ray">
+      <always_on>true</always_on>
+      <update_rate>15.0</update_rate>
+      <visualize>false</visualize>
+      <pose>0 0 0 0 0 0</pose>
+      <ray>
+        <scan>
+          <horizontal>
+            <samples>720</samples>
+            <resolution>1</resolution>
+            <min_angle>${-pi_tcpa}</min_angle>
+            <max_angle>${pi_tcpa}</max_angle>
+          </horizontal>
+        </scan>
+        <range>
+          <min>0.12</min>
+          <max>15.0</max>
+          <resolution>0.01</resolution>
+        </range>
+        <noise>
+          <type>gaussian</type>
+          <mean>0.0</mean>
+          <stddev>0.005</stddev>
+        </noise>
+      </ray>
+      <plugin name="nav_scan_plugin" filename="libgazebo_ros_ray_sensor.so">
+        <ros>
+          <remapping>~/out:=/scan_nav</remapping>
+        </ros>
+        <output_type>sensor_msgs/LaserScan</output_type>
+        <frame_name>nav_scan_frame</frame_name>
+      </plugin>
+    </sensor>
+  </gazebo>
   <xacro:unless value="${lidar_backend == 'livox_plugin'}">
     <gazebo reference="livox_frame">
